File: electronics/signal_generator.sch (EAGLE design)
At the start: 8 parts, among them IC1 LM386N-1

Commit message: increase size of routes and pads
Parts:
- R1, R2, R3, R4: device adafruit:R-US_0204/2V -> adafruit:R-US_0204/7
