File: electronics/terminals.brd (EAGLE design)
At the start: 101.7 x 76.1 mm, 10 parts, among them IC2 L293D, X1 1751303, X2 1751303, X3 1751303, X4 1751303, X5 1751303

Commit message: Add additional vias to the board layout
Any traces that need to connect to the pins of an IC (arduino, GPS or
motor driver) need to do so on the bottom layer. So any traces
that are on the top layer need to be routed through a via to the
bottom layer.
Parts:
- removed U$2: ADALOGGER_M0, Adalogger_32u4:BOARD
- added M0: Adalogger M0, Adalogger_32u4:BOARD
- moved R1 2.30 mm to (19.1, 85.1)
- moved X2 2.30 mm to (91.7, 73.2)
- moved X3 2.30 mm to (81.0, 93.7)
- moved X5 2.30 mm to (50.6, 93.7)
- moved X4 2.30 mm to (91.7, 42.4)
- moved IC2 2.30 mm to (73.5, 73.5)
- moved R5 2.30 mm to (12.7, 85.1)
- moved X1 2.30 mm to (20.1, 93.7)
- moved U$1 2.30 mm to (50.4, 44.8)
Connections:
- removed net N$32: IC2.2, U$2.10
- removed net N$33: IC2.7, U$2.9/A7
- new net L293_1A: IC2.2, M0.10
- new net L293_2A: IC2.7, M0.9/A7
- net 3V3: now also M0.3V; no longer U$2.3V
- net 5V: now also M0.5V; no longer U$2.5V
- net GND: now also M0.GND1; no longer U$2.GND1
- net GPS_RX: now also M0.1/TX; no longer U$2.1/TX
- net GPS_TX: now also M0.0/RX; no longer U$2.0/RX
- net N$28: now also M0.13; no longer U$2.13
- net N$30: now also M0.12; no longer U$2.12
- net NEOPIXEL_SIG: now also M0.18/A4; no longer U$2.18/A4
- net SCL: now also M0.21/SCL; no longer U$2.21/SCL
- net SDA: now also M0.20/SDA; no longer U$2.20/SDA
- net SW_1_2_SIG: now also M0.11; no longer U$2.11
- net SW_3_4_SIG: now also M0.19/A5; no longer U$2.19/A5
- net SW_5_6_SIG: now also M0.6; no longer U$2.6
- net SW_7_8_SIG: now also M0.5; no longer U$2.5
- net THERM_1_SIG: now also M0.14/A0; no longer U$2.14/A0
- net THERM_2_SIG: now also M0.15/A1; no longer U$2.15/A1
- net THERM_3_SIG: now also M0.16/A2; no longer U$2.16/A2
Routing:
- net L293_2A: track 0.00 -> 85.9 mm, vias 0 -> 2
- net N$33: track 81.2 -> 0.00 mm
- net L293_1A: track 0.00 -> 72.7 mm, vias 0 -> 2
- net N$32: track 66.6 -> 0.00 mm
- net MOTOR_1_NEG: track 103.1 -> 125.7 mm, vias 0 -> 2
- net GND: track 338.4 -> 324.5 mm, vias 0 -> 2
- net SCL: track 63.7 -> 69.4 mm, vias 0 -> 1
- net MOTOR_2_POS: track 105.3 -> 110.9 mm
- net NEOPIXEL_SIG: track 62.8 -> 66.7 mm
- net MOTOR_1_POS: track 113.4 -> 117.2 mm
- net 5V: track 174.2 -> 170.5 mm, vias 0 -> 3
- net SW_1_2_SIG: track 104.4 -> 107.9 mm
- net MOTOR_2_NEG: track 102.5 -> 104.0 mm
- net 3V3: track 281.4 -> 280.7 mm, vias 0 -> 1
- net N$28: track 71.0 -> 71.5 mm, vias 0 -> 2
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Other:
- board text added: "Adalogger M0"

Commit message: increase size of routes and pads
Connections:
- net 5V: now also IC2.1
Routing:
- net MOTOR_1_POS: track 117.2 -> 74.7 mm, vias 0 -> 2
- net 3V3: track 280.7 -> 245.8 mm
- net SW_1_2_SIG: track 107.9 -> 87.8 mm, vias 0 -> 2
- net MOTOR_1_NEG: track 125.7 -> 141.0 mm
- net 5V: track 170.5 -> 180.6 mm, vias 3 -> 4
- net GPS_TX: track 19.5 -> 29.3 mm, vias 1 -> 2
- net GND: track 324.5 -> 318.3 mm
- net GPS_RX: track 24.7 -> 30.6 mm, vias 1 -> 2
- net SCL: track 69.4 -> 73.6 mm
- net SDA: track 62.6 -> 66.0 mm
- net N$28: track 71.5 -> 74.0 mm
- net L293_2A: track 85.9 -> 87.1 mm
- net L293_1A: track 72.7 -> 73.7 mm
- net MOTOR_2_POS: track 110.9 -> 110.3 mm
- net THERM_2_SIG: track 113.4 -> 112.9 mm

Commit message: move all traces except vias to bottom layer
Parts:
- R1, R5: device adafruit:0204V -> adafruit:0204/7
- moved R1 5.42 mm to (16.5, 80.3), turned to 90 degrees
- moved R5 5.10 mm to (10.8, 80.4), turned to 270 degrees
Routing:
- net GND: track 318.3 -> 363.7 mm, vias 2 -> 13
- net 3V3: track 245.8 -> 229.1 mm, vias 1 -> 6
- net SDA: track 66.0 -> 73.1 mm, vias 1 -> 2
- net SCL: track 73.6 -> 80.3 mm, vias 1 -> 2
- net MOTOR_2_POS: track 110.3 -> 105.0 mm
- net MOTOR_2_NEG: track 104.0 -> 99.1 mm
- net MOTOR_1_POS: track 74.7 -> 78.5 mm
- net THERM_1_SIG: track 126.5 -> 124.6 mm
- net 5V: track 180.6 -> 179.1 mm
- net THERM_2_SIG: track 112.9 -> 112.2 mm
Other:
- board size 101.7 x 76.1 mm -> 101.6 x 76.2 mm
