File: electronics/terminals.sch (EAGLE design)
At the start: 10 parts, among them IC2 L293D, X1 1751303, X2 1751303, X3 1751303, X4 1751303, X5 1751303

Commit message: Add additional vias to the board layout
Any traces that need to connect to the pins of an IC (arduino, GPS or
motor driver) need to do so on the bottom layer. So any traces
that are on the top layer need to be routed through a via to the
bottom layer.
Parts:
- M0: value ADALOGGER_M0 -> Adalogger M0
- renumbered U$2 to M0
Connections:
- net N$32 renamed L293_1A
- net N$33 renamed L293_2A
Changed lines of the file:
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@@
 <part name="R5" library="adafruit" library_urn="urn:adsk.eagle:library:420" deviceset="R-US_" device="0204/2V" package3d_urn="urn:adsk.eagle:package:6240630/1" value="1 kΩ"/>
 <part name="U$1" library="Adalogger_32u4" deviceset="GPS" device=""/>
-<part name="U$2" library="Adalogger_32u4" deviceset="ADALOGGER_M0" device=""/>
 <part name="X5" library="con-phoenix-350" library_urn="urn:adsk.eagle:library:174" deviceset="1751303" device="" package3d_urn="urn:adsk.eagle:package:9408/1"/>
+<part name="M0" library="Adalogger_32u4" deviceset="ADALOGGER_M0" device="" value="Adalogger M0"/>
 </parts>
 <sheets>
@@
 </instance>
 <instance part="U$1" gate="G$1" x="53.34" y="-43.18" smashed="yes" rot="R180"/>
-<instance part="U$2" gate="G$1" x="78.74" y="99.06" smashed="yes"/>
 <instance part="X5" gate="-1" x="68.58" y="127" smashed="yes" rot="R90">
 <attribute name="NAME" x="69.469" y="128.27" size="1.778" layer="95" rot="R90"/>
@@
 <attribute name="NAME" x="122.809" y="128.27" size="1.778" layer="95" rot="R90"/>
 </instance>
+<instance part="M0" gate="G$1" x="78.74" y="99.06" smashed="yes"/>
 </instances>
 <busses>
@@
 <pinref part="IC2" gate="G$1" pin="4A"/>
 <wire x1="144.78" y1="-15.24" x2="114.3" y2="-15.24" width="0.1524" layer="91"/>
-<pinref part="U$2" gate="G$1" pin="13"/>
+<pinref part="M0" gate="G$1" pin="13"/>
 </segment>
 </net>
@@
 <wire x1="142.24" y1="48.26" x2="142.24" y2="-40.64" width="0.1524" layer="91"/>
 <wire x1="142.24" y1="-40.64" x2="114.3" y2="-40.64" width="0.1524" layer="91"/>
-<pinref part="U$2" gate="G$1" pin="12"/>
-</segment>
-</net>
-<net name="N$32" class="0">
+<pinref part="M0" gate="G$1" pin="12"/>
+</segment>
+</net>
+<net name="L293_1A" class="0">
 <segment>
 <wire x1="124.46" y1="38.1" x2="137.16" y2="38.1" width="0.1524" layer="91"/>
@@
 <pinref part="IC2" gate="G$1" pin="1A"/>
 <wire x1="78.74" y1="-15.24" x2="83.82" y2="-15.24" width="0.1524" layer="91"/>
-<pinref part="U$2" gate="G$1" pin="10"/>
-</segment>
-</net>
-<net name="N$33" class="0">
+<pinref part="M0" gate="G$1" pin="10"/>
+</segment>
+</net>
+<net name="L293_2A" class="0">
 <segment>
 <wire x1="124.46" y1="33.02" x2="129.54" y2="33.02" width="0.1524" layer="91"/>
@@
 <pinref part="IC2" gate="G$1" pin="2A"/>
 <wire x1="76.2" y1="-40.64" x2="83.82" y2="-40.64" width="0.1524" layer="91"/>
-<pinref part="U$2" gate="G$1" pin="9"/>
+<pinref part="M0" gate="G$1" pin="9"/>
 </segment>
 </net>
@@
 <pinref part="IC2" gate="G$1" pin="VCC1"/>
 <wire x1="132.08" y1="-10.16" x2="116.84" y2="-10.16" width="0.1524" layer="91"/>
-<pinref part="U$2" gate="G$1" pin="VBUS/USB"/>
 <wire x1="116.84" y1="-10.16" x2="114.3" y2="-10.16" width="0.1524" layer="91"/>
 <pinref part="IC2" gate="G$1" pin="VCC2"/>
@@
 <wire x1="33.02" y1="81.28" x2="55.88" y2="81.28" width="0.1524" layer="91"/>
 <junction x="55.88" y="81.28"/>
+<pinref part="M0" gate="G$1" pin="VBUS/USB"/>
 </segment>
 </net>
@@
 <wire x1="147.32" y1="20.32" x2="147.32" y2="12.7" width="0.1524" layer="91"/>
 <junction x="147.32" y="12.7"/>
-<pinref part="U$2" gate="G$1" pin="20/SDA"/>
+<pinref part="M0" gate="G$1" pin="20/SDA"/>
 </segment>
 </net>
@@
 <wire x1="152.4" y1="20.32" x2="152.4" y2="17.78" width="0.1524" layer="91"/>
 <junction x="152.4" y="17.78"/>
-<pinref part="U$2" gate="G$1" pin="21/SCL"/>
+<pinref part="M0" gate="G$1" pin="21/SCL"/>
 </segment>
 </net>
@@
 <wire x1="63.5" y1="-25.4" x2="63.5" y2="22.86" width="0.1524" layer="91"/>
 <wire x1="63.5" y1="22.86" x2="73.66" y2="22.86" width="0.1524" layer="91"/>
-<pinref part="U$2" gate="G$1" pin="0/RX"/>
+<pinref part="M0" gate="G$1" pin="0/RX"/>
 </segment>
 </net>
@@
 <wire x1="60.96" y1="-22.86" x2="60.96" y2="17.78" width="0.1524" layer="91"/>
 <wire x1="60.96" y1="17.78" x2="73.66" y2="17.78" width="0.1524" layer="91"/>
-<pinref part="U$2" gate="G$1" pin="1/TX"/>
+<pinref part="M0" gate="G$1" pin="1/TX"/>
 </segment>
 </net>
@@
 <junction x="68.58" y="83.82"/>
 <junction x="68.58" y="106.68"/>
-<pinref part="U$2" gate="G$1" pin="3V"/>
 <wire x1="40.64" y1="106.68" x2="68.58" y2="106.68" width="0.1524" layer="91"/>
 <pinref part="X5" gate="-6" pin="K"/>
@@
 <wire x1="33.02" y1="104.14" x2="40.64" y2="104.14" width="0.1524" layer="91"/>
 <wire x1="40.64" y1="104.14" x2="40.64" y2="106.68" width="0.1524" layer="91"/>
+<pinref part="M0" gate="G$1" pin="3V"/>
 </segment>
 </net>
@@
 <wire x1="43.18" y1="111.76" x2="129.54" y2="111.76" width="0.1524" layer="91"/>
 <wire x1="129.54" y1="111.76" x2="129.54" y2="43.18" width="0.1524" layer="91"/>
-<pinref part="U$2" gate="G$1" pin="11"/>
 <wire x1="129.54" y1="43.18" x2="124.46" y2="43.18" width="0.1524" layer="91"/>
 <pinref part="X2" gate="-4" pin="K"/>
@@
 <wire x1="43.18" y1="12.7" x2="38.1" y2="12.7" width="0.1524" layer="91"/>
 <junction x="38.1" y="12.7"/>
+<pinref part="M0" gate="G$1" pin="11"/>
 </segment>
 </net>
 <net name="THERM_3_SIG" class="0">
 <segment>
-<pinref part="U$2" gate="G$1" pin="16/A2"/>
 <pinref part="X4" gate="-7" pin="K"/>
 <wire x1="58.42" y1="58.42" x2="73.66" y2="58.42" width="0.1524" layer="91"/>
 <wire x1="33.02" y1="96.52" x2="58.42" y2="96.52" width="0.1524" layer="91"/>
 <wire x1="58.42" y1="96.52" x2="58.42" y2="58.42" width="0.1524" layer="91"/>
+<pinref part="M0" gate="G$1" pin="16/A2"/>
 </segment>
 </net>
@@
 <segment>
 <wire x1="60.96" y1="116.84" x2="60.96" y2="63.5" width="0.1524" layer="91"/>
-<pinref part="U$2" gate="G$1" pin="15/A1"/>
 <wire x1="60.96" y1="63.5" x2="73.66" y2="63.5" width="0.1524" layer="91"/>
 <pinref part="X5" gate="-4" pin="K"/>
 <wire x1="91.44" y1="124.46" x2="91.44" y2="116.84" width="0.1524" layer="91"/>
 <wire x1="91.44" y1="116.84" x2="60.96" y2="116.84" width="0.1524" layer="91"/>
+<pinref part="M0" gate="G$1" pin="15/A1"/>
 </segment>
 </net>
@@
 <pinref part="X5" gate="-7" pin="K"/>
 <wire x1="114.3" y1="119.38" x2="114.3" y2="124.46" width="0.1524" layer="91"/>
-<pinref part="U$2" gate="G$1" pin="14/A0"/>
 <wire x1="63.5" y1="119.38" x2="63.5" y2="68.58" width="0.1524" layer="91"/>
 <wire x1="63.5" y1="68.58" x2="73.66" y2="68.58" width="0.1524" layer="91"/>
+<pinref part="M0" gate="G$1" pin="14/A0"/>
 </segment>
 </net>
@@
 <wire x1="63.5" y1="-30.48" x2="68.58" y2="-30.48" width="0.1524" layer="91"/>
 <junction x="68.58" y="-30.48"/>
-<pinref part="U$2" gate="G$1" pin="GND1"/>
 <pinref part="X3" gate="-8" pin="K"/>
 <wire x1="175.26" y1="35.56" x2="172.72" y2="35.56" width="0.1524" layer="91"/>
@@
 <wire x1="33.02" y1="58.42" x2="35.56" y2="58.42" width="0.1524" layer="91"/>
 <junction x="35.56" y="58.42"/>
+<pinref part="M0" gate="G$1" pin="GND1"/>
 </segment>
 </net>
 <net name="SW_3_4_SIG" class="0">
 <segment>
-<pinref part="U$2" gate="G$1" pin="19/A5"/>
 <pinref part="X2" gate="-8" pin="K"/>
 <wire x1="38.1" y1="43.18" x2="33.02" y2="43.18" width="0.1524" layer="91"/>
@@
 <wire x1="73.66" y1="43.18" x2="38.1" y2="43.18" width="0.1524" layer="91"/>
 <junction x="38.1" y="43.18"/>
+<pinref part="M0" gate="G$1" pin="19/A5"/>
 </segment>
 </net>
@@
 <junction x="170.18" y="73.66"/>
 <wire x1="139.7" y1="73.66" x2="139.7" y2="27.94" width="0.1524" layer="91"/>
-<pinref part="U$2" gate="G$1" pin="6"/>
 <wire x1="124.46" y1="27.94" x2="139.7" y2="27.94" width="0.1524" layer="91"/>
+<pinref part="M0" gate="G$1" pin="6"/>
 </segment>
 </net>
@@
 <junction x="170.18" y="43.18"/>
 <wire x1="134.62" y1="43.18" x2="134.62" y2="22.86" width="0.1524" layer="91"/>
-<pinref part="U$2" gate="G$1" pin="5"/>
 <wire x1="134.62" y1="22.86" x2="124.46" y2="22.86" width="0.1524" layer="91"/>
+<pinref part="M0" gate="G$1" pin="5"/>
 </segment>
 </net>
@@
 <wire x1="33.02" y1="50.8" x2="58.42" y2="50.8" width="0.1524" layer="91"/>
 <wire x1="58.42" y1="50.8" x2="58.42" y2="48.26" width="0.1524" layer="91"/>
-<pinref part="U$2" gate="G$1" pin="18/A4"/>
 <wire x1="58.42" y1="48.26" x2="73.66" y2="48.26" width="0.1524" layer="91"/>
-</segment>
-</net>
+<pinref part="M0" gate="G$1" pin="18/A4"/>
+</segment>
+</net>

Commit message: increase size of routes and pads
Connections:
- net 5V: now also IC2.1-2EN
Changed lines of the file:
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@@
 <junction x="55.88" y="81.28"/>
 <pinref part="M0" gate="G$1" pin="VBUS/USB"/>
+<pinref part="IC2" gate="G$1" pin="1-2EN"/>
+<wire x1="83.82" y1="-10.16" x2="83.82" y2="-5.08" width="0.1524" layer="91"/>
+<wire x1="83.82" y1="-5.08" x2="116.84" y2="-5.08" width="0.1524" layer="91"/>
+<wire x1="116.84" y1="-5.08" x2="116.84" y2="-10.16" width="0.1524" layer="91"/>
 </segment>
 </net>

Commit message: move all traces except vias to bottom layer
Parts:
- R1, R5: device adafruit:R-US_0204/2V -> adafruit:R-US_0204/7
Changed lines of the file:
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@@
 <layers>
 <layer number="1" name="Top" color="4" fill="1" visible="no" active="no"/>
-<layer number="2" name="Route2" color="1" fill="3" visible="no" active="no"/>
-<layer number="3" name="Route3" color="4" fill="3" visible="no" active="no"/>
-<layer number="4" name="Route4" color="1" fill="4" visible="no" active="no"/>
-<layer number="5" name="Route5" color="4" fill="4" visible="no" active="no"/>
-<layer number="6" name="Route6" color="1" fill="8" visible="no" active="no"/>
-<layer number="7" name="Route7" color="4" fill="8" visible="no" active="no"/>
-<layer number="8" name="Route8" color="1" fill="2" visible="no" active="no"/>
-<layer number="9" name="Route9" color="4" fill="2" visible="no" active="no"/>
-<layer number="10" name="Route10" color="1" fill="7" visible="no" active="no"/>
-<layer number="11" name="Route11" color="4" fill="7" visible="no" active="no"/>
-<layer number="12" name="Route12" color="1" fill="5" visible="no" active="no"/>
-<layer number="13" name="Route13" color="4" fill="5" visible="no" active="no"/>
-<layer number="14" name="Route14" color="1" fill="6" visible="no" active="no"/>
-<layer number="15" name="Route15" color="4" fill="6" visible="no" active="no"/>
+<layer number="2" name="Route2" color="16" fill="1" visible="no" active="no"/>
+<layer number="3" name="Route3" color="17" fill="1" visible="no" active="no"/>
+<layer number="4" name="Route4" color="18" fill="1" visible="no" active="no"/>
+<layer number="5" name="Route5" color="19" fill="1" visible="no" active="no"/>
+<layer number="6" name="Route6" color="25" fill="1" visible="no" active="no"/>
+<layer number="7" name="Route7" color="26" fill="1" visible="no" active="no"/>
+<layer number="8" name="Route8" color="27" fill="1" visible="no" active="no"/>
+<layer number="9" name="Route9" color="28" fill="1" visible="no" active="no"/>
+<layer number="10" name="Route10" color="29" fill="1" visible="no" active="no"/>
+<layer number="11" name="Route11" color="30" fill="1" visible="no" active="no"/>
+<layer number="12" name="Route12" color="20" fill="1" visible="no" active="no"/>
+<layer number="13" name="Route13" color="21" fill="1" visible="no" active="no"/>
+<layer number="14" name="Route14" color="22" fill="1" visible="no" active="no"/>
+<layer number="15" name="Route15" color="23" fill="1" visible="no" active="no"/>
 <layer number="16" name="Bottom" color="1" fill="1" visible="no" active="no"/>
 <layer number="17" name="Pads" color="2" fill="1" visible="no" active="no"/>
@@
 <part name="X1" library="con-phoenix-350" library_urn="urn:adsk.eagle:library:174" deviceset="1751303" device="" package3d_urn="urn:adsk.eagle:package:9408/1"/>
 <part name="IC2" library="st-microelectronics" library_urn="urn:adsk.eagle:library:368" deviceset="L293D" device="" package3d_urn="urn:adsk.eagle:package:26820/1"/>
-<part name="R1" library="adafruit" library_urn="urn:adsk.eagle:library:420" deviceset="R-US_" device="0204/2V" package3d_urn="urn:adsk.eagle:package:6240630/1" value="1 kΩ"/>
-<part name="R5" library="adafruit" library_urn="urn:adsk.eagle:library:420" deviceset="R-US_" device="0204/2V" package3d_urn="urn:adsk.eagle:package:6240630/1" value="1 kΩ"/>
+<part name="R1" library="adafruit" library_urn="urn:adsk.eagle:library:420" deviceset="R-US_" device="0204/7" package3d_urn="urn:adsk.eagle:package:6240596/1" value="1 kΩ"/>
+<part name="R5" library="adafruit" library_urn="urn:adsk.eagle:library:420" deviceset="R-US_" device="0204/7" package3d_urn="urn:adsk.eagle:package:6240596/1" value="1 kΩ"/>
 <part name="U$1" library="Adalogger_32u4" deviceset="GPS" device=""/>
 <part name="X5" library="con-phoenix-350" library_urn="urn:adsk.eagle:library:174" deviceset="1751303" device="" package3d_urn="urn:adsk.eagle:package:9408/1"/>
